File: Spooky 1 Mainboard/Spooky 1 Mainboard.kicad_sch (KiCad schematic)
At the start: 0 parts

Commit message: Day 2 Progress; Awaiting Journal Entry
Parts:
- added U1: ~, symbol Spooky-1-Symbols:pico
- added U11: ~, symbol GPIO:3_pin
- added U12: L7805, symbol Regulator_Linear:L7805
- added U2, U3, U4, U5: ~, symbol Spooky-1-Symbols:TMC2209
- added U6, U7, U8, U9: ~, symbol GPIO:4_pin
Connections:
- new net: U1.33 (GND), U2.15 (GND), U2.9 (GND), U3.15 (GND), U3.9 (GND), U4.15 (GND), U4.9 (GND), U5.15 (GND), U5.9 (GND)
- new net: U1.36 (3V3(OUT)), U2.10 (VIO), U2.2 (MS1), U2.3 (MS2), U3.10 (VIO), U3.2 (MS1), U3.3 (MS2), U4.10 (VIO), U4.2 (MS1), U4.3 (MS2), U5.10 (VIO), U5.2 (MS1), U5.3 (MS2)
- new net: U1.38 (GND), U11.3 (pin_3), U12.2 (GND)
- new net: U1.40 (VBUS), U12.3 (OUT)
- new net: U4.11 (M2B), U8.1 (pin_1)
- new net: U4.12 (M2A), U8.2 (pin_2)
- new net: U4.13 (M1A), U8.3 (pin_3)
- new net: U4.14 (M1B), U8.4 (pin_4)
- new net: U4.4 (PDN), U4.5 (USART)
- new net: U5.11 (M2B), U9.1 (pin_1)
- new net: U5.12 (M2A), U9.2 (pin_2)
- new net: U5.13 (M1A), U9.3 (pin_3)
- new net: U5.14 (M1B), U9.4 (pin_4)
- new net: U5.4 (PDN), U5.5 (USART)
- new net: U2.11 (M2B), U6.1 (pin_1)
- new net: U2.12 (M2A), U6.2 (pin_2)
- new net: U2.13 (M1A), U6.3 (pin_3)
- new net: U2.14 (M1B), U6.4 (pin_4)
- new net: U2.4 (PDN), U2.5 (USART)
- new net: U11.2 (pin_2), U12.1 (IN)
- new net: U3.11 (M2B), U7.1 (pin_1)
- new net: U3.12 (M2A), U7.2 (pin_2)
- new net: U3.13 (M1A), U7.3 (pin_3)
- new net: U3.14 (M1B), U7.4 (pin_4)
- new net: U3.4 (PDN), U3.5 (USART)
